File: TestboardV2.2a.sch (KiCad schematic (older format))
At the start: 32 parts, among them IC1 BME680, IC2 MAX17048G+, IC3 LTC2954CTS8-1#TRMPBF, J10 Conn_01x04, J12 Conn_01x02, J7 Conn_01x04, J8 Conn_01x02, Q2 DMG2301L, SW2 SW_Push, U15 MCP73831-2-OT

Commit message: Added LDO CE Pullup. JLCPCB files updated
Parts:
- added JP24: SolderJumper_2_Open, Jumper:SolderJumper-2_P1.3mm_Open_RoundedPad1.0x1.5mm, symbol Jumper:SolderJumper_2_Open
Connections:
- net CE: now also JP24.2 (B); no longer D14.1 (K)
- new net: D14.1 (K), JP24.1 (A)
Other:
- note added: "Optional"
Changed lines of the file:
@@
 Wire Wire Line
 	9450 1550 10200 1550
-Wire Wire Line
-	7350 4000 7350 4350
-Text GLabel 7350 4350 3    50   Output ~ 0
+Text GLabel 7350 4900 3    50   Output ~ 0
 CE
 $Comp
@@
 	0    1    1    0
 $EndComp
+Text Notes 6900 3900 0    50   ~ 0
+Optional
+$Comp
+L Jumper:SolderJumper_2_Open JP24
+U 1 1 61782FB8
+P 7350 4600
+F 0 "JP24" V 7304 4668 50  0000 L CNN
+F 1 "SolderJumper_2_Open" V 7395 4668 50  0000 L CNN
+F 2 "Jumper:SolderJumper-2_P1.3mm_Open_RoundedPad1.0x1.5mm" H 7350 4600 50  0001 C CNN
+F 3 "~" H 7350 4600 50  0001 C CNN
+	1    7350 4600
+	0    1    1    0
+$EndComp
+Wire Wire Line
+	7350 4000 7350 4450
+Wire Wire Line
+	7350 4750 7350 4900
 $EndSCHEMATC
