File: TestboardV2.3.sch (KiCad schematic (older format))
At the start: 81 parts, among them J13 USB_C_Receptacle_USB2.0 USB41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, J2 Conn_01x04_MountingPin, J3 Conn_01x04_MountingPin, J4 Conn_01x04_MountingPin, J5 Conn_01x04_MountingPin, J6 Conn_01x04_MountingPin, J9 Conn_01x03, Q1 UMH3N, SW1 SW_Push, U1 ESP32-WROOM-32D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

Commit message: Testboard V2.3
Parts:
- added C24, C25: 10µF, Capacitor_SMD:C_0805_2012Metric, symbol Device:C
Connections:
- net +3V3: now also C25.1
- net +5V: now also C24.1
- net GND: now also C24.2, C25.2
Other:
- moved on the sheet: C11, C9, D15, JP21, R29, R37
Changed lines of the file:
@@
 encoding utf-8
 Sheet 1 3
-Title "Testboard V2.2"
-Date "2021-04-28"
-Rev "V0.1"
+Title "Testboard V2.3"
+Date "2021-12-11"
+Rev "V0.2"
 Comp "Ratamuse"
 Comment1 ""
@@
 Text GLabel 10650 3400 2    50   Input ~ 0
 RST_EN
-Text GLabel 7500 4150 0    50   Input ~ 0
+Text GLabel 7200 4150 0    50   Input ~ 0
 +5V
 $Comp
@@
 $EndComp
 Wire Wire Line
-	8000 4150 8000 4300
-Wire Wire Line
-	8000 4600 8000 4750
+	8100 4150 8100 4300
+Wire Wire Line
+	8100 4600 8100 4750
 $Comp
 L Device:C C9
 U 1 1 5F6315DF
-P 8000 4450
-F 0 "C9" H 8115 4496 50  0000 L CNN
-F 1 "0.1µF" H 8115 4405 50  0000 L CNN
-F 2 "Capacitor_SMD:C_0603_1608Metric" H 8038 4300 50  0001 C CNN
-F 3 "~" H 8000 4450 50  0001 C CNN
-	1    8000 4450
+P 8100 4450
+F 0 "C9" H 8215 4496 50  0000 L CNN
+F 1 "0.1µF" H 8215 4405 50  0000 L CNN
+F 2 "Capacitor_SMD:C_0603_1608Metric" H 8138 4300 50  0001 C CNN
+F 3 "~" H 8100 4450 50  0001 C CNN
+	1    8100 4450
 	1    0    0    -1
 $EndComp
@@
 L power:GND #PWR0112
 U 1 1 5F6315D5
-P 8000 4750
-F 0 "#PWR0112" H 8000 4500 50  0001 C CNN
-F 1 "GND" H 8005 4577 50  0000 C CNN
-F 2 "" H 8000 4750 50  0001 C CNN
-F 3 "" H 8000 4750 50  0001 C CNN
-	1    8000 4750
-	1    0    0    -1
-$EndComp
-$Comp
-L Device:C C11
-U 1 1 5F639961
-P 9700 4450
-F 0 "C11" H 9815 4496 50  0000 L CNN
-F 1 "0.1µF" H 9815 4405 50  0000 L CNN
-F 2 "Capacitor_SMD:C_0603_1608Metric" H 9738 4300 50  0001 C CNN
-F 3 "~" H 9700 4450 50  0001 C CNN
-	1    9700 4450
-	1    0    0    -1
-$EndComp
-$Comp
-L power:GND #PWR0114
-U 1 1 5F63996B
-P 9700 4750
-F 0 "#PWR0114" H 9700 4500 50  0001 C CNN
-F 1 "GND" H 9705 4577 50  0000 C CNN
-F 2 "" H 9700 4750 50  0001 C CNN
-F 3 "" H 9700 4750 50  0001 C CNN
-	1    9700 4750
-	1    0    0    -1
-$EndComp
-Wire Wire Line
-	9700 4600 9700 4750
-Text GLabel 10450 4250 2    50   Output ~ 0
+P 8100 4750
+F 0 "#PWR0112" H 8100 4500 50  0001 C CNN
+F 1 "GND" H 8105 4577 50  0000 C CNN
+F 2 "" H 8100 4750 50  0001 C CNN
+F 3 "" H 8100 4750 50  0001 C CNN
+	1    8100 4750
+	1    0    0    -1
+$EndComp
+Text GLabel 10600 4250 2    50   Output ~ 0
 +3V3
 Text GLabel 800  3350 0    50   Input ~ 0
@@
 	600  2650 600  2600
 Wire Wire Line
-	10150 4250 10450 4250
+	10300 4250 10600 4250
 $Comp
 L Jumper:SolderJumper_2_Open JP21
 U 1 1 611603B3
-P 10150 4500
-F 0 "JP21" V 10104 4568 50  0000 L CNN
-F 1 "SolderJumper_2_Open" V 10195 4568 50  0000 L CNN
-F 2 "Jumper:SolderJumper-2_P1.3mm_Open_RoundedPad1.0x1.5mm" H 10150 4500 50  0001 C CNN
-F 3 "~" H 10150 4500 50  0001 C CNN
-	1    10150 4500
+P 10300 4500
+F 0 "JP21" V 10254 4568 50  0000 L CNN
+F 1 "SolderJumper_2_Open" V 10345 4568 50  0000 L CNN
+F 2 "Jumper:SolderJumper-2_P1.3mm_Open_RoundedPad1.0x1.5mm" H 10300 4500 50  0001 C CNN
+F 3 "~" H 10300 4500 50  0001 C CNN
+	1    10300 4500
 	0    1    1    0
 $EndComp
@@
 L Device:LED D15
 U 1 1 6119BB9E
-P 10150 5150
-F 0 "D15" H 10143 4895 50  0000 C CNN
-F 1 "LED Green" H 10143 4986 50  0000 C CNN
-F 2 "LED_SMD:LED_0603_1608Metric_Castellated" H 10150 5150 50  0001 C CNN
-F 3 "~" H 10150 5150 50  0001 C CNN
-	1    10150 5150
+P 10300 5150
+F 0 "D15" H 10293 4895 50  0000 C CNN
+F 1 "LED Green" H 10293 4986 50  0000 C CNN
+F 2 "LED_SMD:LED_0603_1608Metric_Castellated" H 10300 5150 50  0001 C CNN
+F 3 "~" H 10300 5150 50  0001 C CNN
+	1    10300 5150
 	0    -1   -1   0
 $EndComp
@@
 L Device:R R29
 U 1 1 6119C5BC
-P 10150 4800
-F 0 "R29" V 9943 4800 50  0000 C CNN
-F 1 "10K" V 10034 4800 50  0000 C CNN
-F 2 "Resistor_SMD:R_0603_1608Metric" V 10080 4800 50  0001 C CNN
-F 3 "~" H 10150 4800 50  0001 C CNN
-	1    10150 4800
+P 10300 4800
+F 0 "R29" V 10093 4800 50  0000 C CNN
+F 1 "10K" V 10184 4800 50  0000 C CNN
+F 2 "Resistor_SMD:R_0603_1608Metric" V 10230 4800 50  0001 C CNN
+F 3 "~" H 10300 4800 50  0001 C CNN
+	1    10300 4800
 	-1   0    0    1
 $EndComp
 Wire Wire Line
-	10150 4950 10150 5000
+	10300 4950 10300 5000
 $Comp
 L power:GND #PWR0166
 U 1 1 6124F321
-P 10150 5350
-F 0 "#PWR0166" H 10150 5100 50  0001 C CNN
-F 1 "GND" H 10155 5177 50  0000 C CNN
-F 2 "" H 10150 5350 50  0001 C CNN
-F 3 "" H 10150 5350 50  0001 C CNN
-	1    10150 5350
-	1    0    0    -1
-$EndComp
-Wire Wire Line
-	10150 5300 10150 5350
+P 10300 5350
+F 0 "#PWR0166" H 10300 5100 50  0001 C CNN
+F 1 "GND" H 10305 5177 50  0000 C CNN
+F 2 "" H 10300 5350 50  0001 C CNN
+F 3 "" H 10300 5350 50  0001 C CNN
+	1    10300 5350
+	1    0    0    -1
+$EndComp
+Wire Wire Line
+	10300 5300 10300 5350
 $Comp
 L Device:R R37
 U 1 1 616E1E53
-P 7600 4400
-F 0 "R37" V 7393 4400 50  0000 C CNN
-F 1 "100K" V 7484 4400 50  0000 C CNN
-F 2 "Resistor_SMD:R_0603_1608Metric" V 7530 4400 50  0001 C CNN
-F 3 "~" H 7600 4400 50  0001 C CNN
-	1    7600 4400
+P 7300 4400
+F 0 "R37" V 7093 4400 50  0000 C CNN
+F 1 "100K" V 7184 4400 50  0000 C CNN
+F 2 "Resistor_SMD:R_0603_1608Metric" V 7230 4400 50  0001 C CNN
+F 3 "~" H 7300 4400 50  0001 C CNN
+	1    7300 4400
 	-1   0    0    1
 $EndComp
-Connection ~ 8000 4150
-Wire Wire Line
-	8350 4350 8350 4650
-Wire Wire Line
-	7600 4650 8350 4650
-Connection ~ 8350 4650
-Wire Wire Line
-	8350 4650 8350 4750
-Wire Wire Line
-	7500 4150 7600 4150
-Wire Wire Line
-	7600 4650 7600 4550
-Wire Wire Line
-	7600 4250 7600 4150
-Connection ~ 7600 4150
-Wire Wire Line
-	7600 4150 8000 4150
-Wire Wire Line
-	8000 4150 8450 4150
+Wire Wire Line
+	7200 4150 7300 4150
+Wire Wire Line
+	7300 4650 7300 4550
+Wire Wire Line
+	7300 4250 7300 4150
+Connection ~ 7300 4150
 Wire Wire Line
 	8950 4650 8950 4800
@@
 Wire Wire Line
 	8400 4650 8950 4650
+Connection ~ 10300 4250
+Wire Wire Line
+	10300 4250 10300 4350
+$Sheet
+S 0    8500 3050 2300
+U 6011445D
+F0 "TestboardV2.3a" 50
+F1 "TestboardV2.3a.sch" 50
+$EndSheet
+$Sheet
+S 0    11400 4000 2550
+U 609E7AF1
+F0 "TestboardV2.3b" 50
+F1 "TestboardV2.3b.sch" 50
+$EndSheet
+Connection ~ 9600 4250
+Wire Wire Line
+	9600 4250 10050 4250
+Wire Wire Line
+	9550 4250 9600 4250
+Wire Wire Line
+	9600 4300 9600 4250
 $Comp
 L XC6220B331MR-G:XC6220B331MR-G U13
@@
 $EndComp
 Wire Wire Line
-	9550 4250 9700 4250
-Connection ~ 10150 4250
-Wire Wire Line
-	10150 4250 10150 4350
-Wire Wire Line
-	9700 4300 9700 4250
-Connection ~ 9700 4250
-Wire Wire Line
-	9700 4250 10150 4250
-$Sheet
-S 0    8500 3050 2300
-U 6011445D
-F0 "TestboardV2.2a" 50
-F1 "TestboardV2.2a.sch" 50
-$EndSheet
-$Sheet
-S 0    11400 4000 2550
-U 609E7AF1
-F0 "TestboardV2.2b" 50
-F1 "TestboardV2.2b.sch" 50
-$EndSheet
+	9600 4600 9600 4750
+$Comp
+L power:GND #PWR0114
+U 1 1 5F63996B
+P 9600 4750
+F 0 "#PWR0114" H 9600 4500 50  0001 C CNN
+F 1 "GND" H 9605 4577 50  0000 C CNN
+F 2 "" H 9600 4750 50  0001 C CNN
+F 3 "" H 9600 4750 50  0001 C CNN
+	1    9600 4750
+	1    0    0    -1
+$EndComp
+$Comp
+L Device:C C11
+U 1 1 5F639961
+P 9600 4450
+F 0 "C11" H 9715 4496 50  0000 L CNN
+F 1 "0.1µF" H 9715 4405 50  0000 L CNN
+F 2 "Capacitor_SMD:C_0603_1608Metric" H 9638 4300 50  0001 C CNN
+F 3 "~" H 9600 4450 50  0001 C CNN
+	1    9600 4450
+	1    0    0    -1
+$EndComp
+Wire Wire Line
+	10050 4300 10050 4250
+Wire Wire Line
+	10050 4600 10050 4750
+$Comp
+L power:GND #PWR0161
+U 1 1 61BFC9C6
+P 10050 4750
+F 0 "#PWR0161" H 10050 4500 50  0001 C CNN
+F 1 "GND" H 10055 4577 50  0000 C CNN
+F 2 "" H 10050 4750 50  0001 C CNN
+F 3 "" H 10050 4750 50  0001 C CNN
+	1    10050 4750
+	1    0    0    -1
+$EndComp
+$Comp
+L Device:C C25
+U 1 1 61BFC9D0
+P 10050 4450
+F 0 "C25" H 10165 4496 50  0000 L CNN
+F 1 "10µF" H 10165 4405 50  0000 L CNN
+F 2 "Capacitor_SMD:C_0805_2012Metric" H 10088 4300 50  0001 C CNN
+F 3 "~" H 10050 4450 50  0001 C CNN
+	1    10050 4450
+	1    0    0    -1
+$EndComp
+Connection ~ 10050 4250
+Wire Wire Line
+	10050 4250 10300 4250
+Wire Wire Line
+	8350 4350 8350 4650
+Wire Wire Line
+	7300 4150 7700 4150
+Wire Wire Line
+	7700 4150 7700 4300
+Wire Wire Line
+	7700 4600 7700 4750
+$Comp
+L Device:C C24
+U 1 1 61C7827C
+P 7700 4450
+F 0 "C24" H 7815 4496 50  0000 L CNN
+F 1 "10µF" H 7815 4405 50  0000 L CNN
+F 2 "Capacitor_SMD:C_0805_2012Metric" H 7738 4300 50  0001 C CNN
+F 3 "~" H 7700 4450 50  0001 C CNN
+	1    7700 4450
+	1    0    0    -1
+$EndComp
+$Comp
+L power:GND #PWR0162
+U 1 1 61C78286
+P 7700 4750
+F 0 "#PWR0162" H 7700 4500 50  0001 C CNN
+F 1 "GND" H 7705 4577 50  0000 C CNN
+F 2 "" H 7700 4750 50  0001 C CNN
+F 3 "" H 7700 4750 50  0001 C CNN
+	1    7700 4750
+	1    0    0    -1
+$EndComp
+Connection ~ 7700 4150
+Wire Wire Line
+	7700 4150 8100 4150
+Connection ~ 8100 4150
+Wire Wire Line
+	8100 4150 8450 4150
+Wire Wire Line
+	7300 4650 8350 4650
+Connection ~ 8350 4650
+Wire Wire Line
+	8350 4650 8350 4750
 $EndSCHEMATC
