File: TestboardV2.3a.sch (KiCad schematic (older format))
At the start: 33 parts, among them IC1 BME680, IC2 MAX17048G+, IC3 LTC2954CTS8-1#TRMPBF, J10 Conn_01x04, J12 Conn_01x02, J7 Conn_01x04, J8 Conn_01x02, Q2 DMG2301L, SW2 SW_Push, U15 MCP73831-2-OT

Commit message: Testboard V2.3
Parts:
- removed C12: 0.1µF, Capacitor_SMD:C_0603_1608Metric, symbol Device:C
- removed C13: 1µF, Capacitor_SMD:C_0603_1608Metric, symbol Device:C
- removed IC1: BME680, Empreintes:BME680, symbol BME680:BME680
- added C20: 0.1µF, Capacitor_SMD:C_0603_1608Metric, symbol Device:C
- added IC6: SHT41-AD1B-R3, Empreintes:SHT41AD1BR3, symbol SHT41-AD1B-R3:SHT41-AD1B-R3
- C10, C8: value TBD -> 0.150µF
- JP24: renamed from JP?; footprint (none) -> Jumper:SolderJumper-2_P1.3mm_Open_RoundedPad1.0x1.5mm
Connections:
- net +3V3: now also C20.1, IC6.3 (VDD)
- net GND: now also J12.1 (Pin_1), C20.2, IC6.4 (VSS); no longer J12.2 (Pin_2)
- net SCL: now also IC6.2 (SCL)
- net SDA: now also IC6.1 (SDA)
- net VBAT: now also J12.2 (Pin_2), J8.2 (Pin_2); no longer J12.1 (Pin_1), J8.1 (Pin_1)
- net VBAT-: now also J8.1 (Pin_1); no longer J8.2 (Pin_2)
Other:
- note added: "ONT & PDT capacitor calculation: \nCPDT = 1.56 × 10-4 [μF/ms] • (tPDT – 1ms)\nCONT = 1.56 × 10–4 [μF/ms] • (tONT – 1ms)\n\n0.150µF =962ms +y a fixed internal 64ms delay (t PD,MIN) or 32ms (tDB,ON)"
- moved on the sheet: R15, R17
