File: TestboardV2.3b.sch (KiCad schematic (older format))
At the start: 31 parts, among them IC4 CN3791, IC5 FS312F-G, J11 Conn_01x02, Q3 AO3401A, Q4 FS8205, Q5 AO3400, SW4 SW_Push

Commit message: Testboard V2.3
Parts:
- removed Q5: AO3400, Empreintes:SOT95P280X125-3N, symbol AO3400:AO3400
- removed R32: 1.2K, Resistor_SMD:R_0603_1608Metric, symbol Device:R
- removed SW4: SW_Push, Empreintes:PTS636SL43SMTRLFS, symbol Switch:SW_Push
- R23: value 140K -> 30K
- R25: value 2K -> 10K
- R28: value 0.05R -> 0.24R
- renumbered C19 to C12, C14 to C13, C21 to C14, C22 to C19, C23 to C21, C25 to C22, C26 to C23, D9 to D10, D10 to D11, D11 to D12, D12 to D13, D13 to D8, D8 to D9, IC4 to IC1, IC5 to IC4, J11 to J1
Connections:
- net VBAT-: now also C27.2, IC4.6 (GND), Q4.1 (S1)
- net Vsolar: now also Q3.2 (S); no longer Q3.3 (D)
- net at D13.2: now also Q3.3 (D); no longer Q3.2 (S)
Other:
- note added: "1/The maximum power point voltage is decided\nby the following equation:\n\nVMPPT=1.205x(1+R23/R27)\n\n2/Charge current setting\n\nThe full-scale charge current, namely the charge current in \nconstant current mode, is decided by the following formula:\n\nICH= 120mV/R28\n\n500mA=0.24 ohm\n250mA=0.48 ohm\n125mA=0.96 ohm"
- note removed: "1/The maximum power point voltage is decided\nby the following equation:\n\nVMPPT=1.205x(1+R23/R27)\n\n2/Charge current setting\n\nThe full-scale charge current, namely the charge current in \nconstant current mode, is decided by the following formula:\n\nICH= 120mV/R28"
